File: PCBs/4 Axis FOC Stepper Driver/4 Axis FOC Stepper Driver.kicad_sch (KiCad schematic)
At the start: 18 parts, among them J1 USB_C_Receptacle_USB2.0_16P, SW1 RESET, SW2 BOOT, U1 ESP32-S3-WROOM-1, U2 AMS1117-3.3, U3 TSV994, U6 TSV994

Commit message: Hopefully finally chose a motor driver
Other:
- removed sheet Motor 3
- removed sheet Motor 4
Changed lines of the file:
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@@
-	)
-	(sheet
-		(at 248.92 68.58)
-		(size 12.7 3.81)
-		(fields_autoplaced yes)
-		(stroke
-			(width 0.1524)
-			(type solid)
-		)
-		(fill
-			(color 0 0 0 0.0000)
-		)
-		(property "Sheetname" "Motor 4"
-			(at 248.92 67.8684 0)
-			(effects
-				(font
-					(size 1.27 1.27)
-				)
-				(justify left bottom)
-			)
-		)
-		(property "Sheetfile" "m4.kicad_sch"
-			(at 248.92 72.9746 0)
-			(effects
-				(font
-					(size 1.27 1.27)
-				)
-				(justify left top)
-			)
-		)
-		(instances
-			(project "4 Axis FOC Stepper Driver"
-				(path "/e91d8688-a49f-47f5-b4fd-09a07252fdc2"
-					(page "5")
-				)
-			)
-		)
 	)
 	(sheet
@@
 				)
 			)
-		)
-	)
-	(sheet
-		(at 248.92 59.69)
-		(size 12.7 3.81)
-		(fields_autoplaced yes)
-		(stroke
-			(width 0.1524)
-			(type solid)
-		)
-		(fill
-			(color 0 0 0 0.0000)
-		)
-		(property "Sheetname" "Motor 3"
-			(at 248.92 58.9784 0)
-			(effects
-				(font
-					(size 1.27 1.27)
-				)
-				(justify left bottom)
-			)
-		)
-		(property "Sheetfile" "m3.kicad_sch"
-			(at 248.92 64.0846 0)
-			(effects
-				(font
-					(size 1.27 1.27)
-				)
-				(justify left top)
-			)
-		)
-		(instances
-			(project "4 Axis FOC Stepper Driver"
-				(path "/e91d8688-a49f-47f5-b4fd-09a07252fdc2"
-					(page "4")
-				)
-			)
