File: PCBs/Integrated FOC Stepper Driver/Integrated FOC Stepper Driver.kicad_pcb (KiCad board)
At the start: 6 copper layers, 40 x 40 mm, 65 parts, among them J1 INPUT, J2 USB C Receptacle, J3 OUTPUT, J4 MOTOR, J5 Conn_01x02, SW1 BOOT, SW2 RESET, U1 PJ54M50SE, U2 PJ9500M33SA, U3 RP2040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

Commit message: Start RP2350 design
Parts:
- C16, C20: value 1u -> 1uF
- moved D3 55.8 mm to (90.7, 57.0), turned to 0 degrees
- moved C25 54.3 mm to (82.8, 52.2), turned to 0 degrees
- moved U1 53.3 mm to (95.7, 57.0), turned to 0 degrees
- moved Y1 52.8 mm to (95.5, 39.5)
- moved C1 48.1 mm to (86.2, 46.5), turned to 0 degrees
- moved R14 46.3 mm to (83.0, 40.3), turned to 0 degrees
- moved C3 45.9 mm to (74.2, 46.3), turned to 0 degrees
- moved C4 44.0 mm to (86.2, 51.6)
- moved U3 42.9 mm to (92.9, 49.9), turned to 0 degrees
- moved R1 41.2 mm to (74.2, 38.3), turned to 0 degrees
- moved U2 41.2 mm to (90.7, 61.6), turned to 0 degrees
- moved R16 41.1 mm to (83.0, 44.3), turned to 0 degrees
- moved R15 41.0 mm to (83.0, 42.3), turned to 0 degrees
- moved R5 40.0 mm to (77.1, 38.3), turned to 0 degrees
- moved R2 39.5 mm to (74.2, 40.3), turned to 0 degrees
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Routing:
- net +5V: track 132.2 -> 0.00 mm, vias 4 -> 0
- net /CAN_H: track 39.5 -> 0.00 mm, vias 2 -> 0
- net Net-(D1-DOUT): track 37.3 -> 0.00 mm, vias 2 -> 0
- net /CAN_L: track 33.5 -> 0.00 mm, vias 2 -> 0
- net /B_CURRENT: track 29.1 -> 0.00 mm, vias 4 -> 0
- net Net-(U1-VOUT): track 24.4 -> 0.00 mm, vias 2 -> 0
- net /USB_DP: track 23.5 -> 0.00 mm
- net /RUN: track 23.1 -> 0.00 mm, vias 2 -> 0
- net /USB_DN: track 23.0 -> 0.00 mm
- net /A_CURRENT: track 23.0 -> 0.00 mm, vias 5 -> 0
- net /VUSB: track 22.4 -> 0.00 mm, vias 2 -> 0
- net +3.3V: track 21.6 -> 0.00 mm, vias 21 -> 0
- net /CAN_RX: track 20.3 -> 0.00 mm, vias 2 -> 0
- net +1V1: track 19.2 -> 0.00 mm, vias 3 -> 0
- net /A1_PWM: track 18.9 -> 0.00 mm
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- removed copper zone on F.Cu, net +3.3V
- removed copper zone on In1.Cu, net +3.3V
- removed copper zone on B.Cu, net GND
- removed copper zone on F.Cu, net GND
- removed copper zone on In2.Cu, net GND
- removed copper zone on In4.Cu, net GND
- removed copper zone on In3.Cu, net VBUS
Other:
- board text removed: "+3.3V"
- board text removed: "GND"
- board text removed: "VBUS"
